Commit message: Patch 1 -- Ported URDF to PyBullet!
Next Steps:
- Move Vector Forward in PyBullet
- Lift arm in PyBullet

Signed-off-by: Mihir <Mihir_Parekh@student.uml.edu>

File: urdf/vector.urdf (robot description, URDF)
Before this commit: robot vector, 17 links, 16 joints
Links:
- removed link camera_link
- removed link drop_fl
- removed link drop_fr
- removed link drop_rl
- removed link drop_rr
- removed link imu
- removed link tof_link
Joints:
- removed joint drop_fl_joint
- removed joint drop_fr_joint
- removed joint drop_rl_joint
- removed joint drop_rr_joint
- removed joint head_camera_joint
- removed joint imu_joint
- removed joint tof_joint
- joint front_left_wheel_joint: limit (none) -> lower=-1000 upper=1000 effort=2.0 velocity=15.23; type fixed -> revolute
- joint front_right_wheel_joint: limit (none) -> lower=-1000 upper=1000 effort=2.0 velocity=15.23; type fixed -> revolute
- joint rear_left_wheel_joint: limit (none) -> lower=-1000 upper=1000 effort=2.0 velocity=22.24; type fixed -> revolute
- joint rear_right_wheel_joint: limit (none) -> lower=-1000 upper=1000 effort=2.0 velocity=22.24; type fixed -> revolute
